File: kicad/HWSRedirector.kicad_sch (KiCad schematic)
At the start: 7 parts, among them J1 12V External, K2 FINDER-22.32, SW1 HWS Switch, U1 WeMos C3

Commit message: Updated the schematic
Parts:
- SW1: value HWS Switch -> HWS Switch - May not be needed
- U1: value WeMos C3 -> WeMos C3 or other WiFi Enabled ESP32
Connections:
- net at U2. (Main): no longer K2.1
- net at R1. (vcc): now also U1.10
- new net: K2.11, K2.21, SW1.1 (A)
- new net: R1. (vcc), Reg2. (DC-), U1. (GND)
- new net: R1. (vcc), Reg2. (DC-), U1.VBUS
- now unconnected: U2. (Main)
Other:
- note added: "2 Pole 32A MCB i.e. NHP MOD 6232"
Changed lines of the file:
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@@
-    (stroke (width 0) (type default))
-  )
-  (wire (pts (xy 85.09 81.28) (xy 86.36 81.28))
     (stroke (width 0) (type default))
   )
@@
     (stroke (width 0) (type default))
   )
-  (wire (pts (xy 72.39 72.39) (xy 72.39 81.28))
-    (stroke (width 0) (type default))
-  )
   (wire (pts (xy 76.2 109.1981) (xy 76.2 109.22))
     (stroke (width 0) (type default))
@@
     (stroke (width 0) (type default))
   )
-  (wire (pts (xy 93.98 96.52) (xy 93.98 127))
-    (stroke (width 0) (type default))
-  )
-  (wire (pts (xy 72.39 81.28) (xy 71.12 81.28))
+  (wire (pts (xy 93.98 106.68) (xy 93.98 127))
+    (stroke (width 0) (type default))
+  )
+  (wire (pts (xy 73.66 91.44) (xy 71.12 91.44))
     (stroke (width 0) (type default))
   )
@@
     (stroke (width 0) (type default))
   )
-  (wire (pts (xy 83.82 96.52) (xy 83.82 109.22))
+  (wire (pts (xy 83.82 106.68) (xy 83.82 109.22))
     (stroke (width 0) (type default))
   )
@@
     (stroke (width 0) (type default))
   )
+  (polyline (pts (xy 73.66 77.47) (xy 76.2 73.66))
+    (stroke (width 0.75) (type default))
+  )
   (wire (pts (xy 76.2 109.22) (xy 78.74 109.22))
     (stroke (width 0) (type default))
@@
     (stroke (width 0) (type default))
   )
+  (wire (pts (xy 73.66 55.88) (xy 73.66 73.66))
+    (stroke (width 0) (type default))
+  )
   (wire (pts (xy 170.18 54.61) (xy 136.7307 54.61))
     (stroke (width 0) (type default))
   )
-  (wire (pts (xy 85.09 72.39) (xy 85.09 81.28))
-    (stroke (width 0) (type default))
-  )
   (wire (pts (xy 113.03 111.4946) (xy 113.03 109.22))
     (stroke (width 0) (type default))
@@
     (stroke (width 0) (type default))
   )
-  (wire (pts (xy 73.66 109.1981) (xy 73.66 96.52))
+  (wire (pts (xy 73.66 109.1981) (xy 73.66 106.68))
+    (stroke (width 0) (type default))
+  )
+  (wire (pts (xy 86.36 77.47) (xy 86.36 91.44))
     (stroke (width 0) (type default))
   )
@@
     (stroke (width 0) (type default))
   )
-  (wire (pts (xy 93.98 65.3946) (xy 93.98 81.28))
-    (stroke (width 0) (type default))
+  (wire (pts (xy 93.98 65.3946) (xy 93.98 91.44))
+    (stroke (width 0) (type default))
+  )
+  (polyline (pts (xy 86.36 77.47) (xy 88.9 73.66))
+    (stroke (width 0.75) (type default))
+  )
+  (wire (pts (xy 73.66 77.47) (xy 73.66 91.44))
+    (stroke (width 0) (type default))
+  )
+  (wire (pts (xy 86.36 55.88) (xy 86.36 73.66))
+    (stroke (width 0) (type default))
+  )
+  (rectangle (start 68.58 64.77) (end 91.44 83.82)
+    (stroke (width 0) (type default))
+    (fill (type none))
   )
   (text "5V DC Out" (at 138.43 69.85 0)
@@
     (effects (font (size 3 3) bold) (justify left bottom))
   )
+  (text "2 Pole 32A MCB\ni.e. NHP MOD 6232" (at 49.53 76.2 0)
+    (effects (font (size 1.27 1.27)) (justify left bottom))
+  )
   (text "12V DC in" (at 138.43 114.3 0)
     (effects (font (size 1.27 1.27) bold) (justify left bottom))
@@
     (effects (font (size 3 3) (thickness 0.6) bold) (justify left bottom))
   )
-  (symbol (lib_name "FINDER-30.22_1") (lib_id "Relay:FINDER-30.22") (at 83.82 88.9 0) (mirror y) (unit 1)
-    (in_bom yes) (on_board yes) (dnp no)
-    (property "Reference" "K2" (at 67.818 88.2563 0)
-      (effects (font (size 1.27 1.27)) (justify left))
-    )
-    (property "Value" "FINDER-22.32" (at 64.6888 92.4767 0)
-      (effects (font (size 1.27 1.27)) (justify left))
-    )
-    (property "Footprint" "Relay_THT:Relay_DPDT_Finder_30.22" (at 49.53 89.662 0)
-      (effects (font (size 1.27 1.27)) hide)
-    )
-    (property "Datasheet" "http://gfinder.findernet.com/assets/Series/354/S30EN.pdf" (at 83.82 88.9 0)
+  (symbol (lib_id "Relay:FINDER-30.22") (at 83.82 99.06 0) (mirror y) (unit 1)
+    (in_bom yes) (on_board yes) (dnp no)
+    (property "Reference" "K2" (at 58.42 101.6 0)
+      (effects (font (size 1.27 1.27)) (justify left))
+    )
+    (property "Value" "FINDER-22.32" (at 64.77 99.06 0)
+      (effects (font (size 1.27 1.27)) (justify left))
+    )
+    (property "Footprint" "Relay_THT:Relay_DPDT_Finder_30.22" (at 118.11 99.822 0)
+      (effects (font (size 1.27 1.27)) hide)
+    )
+    (property "Datasheet" "http://gfinder.findernet.com/assets/Series/354/S30EN.pdf" (at 83.82 99.06 0)
+      (effects (font (size 1.27 1.27)) hide)
+    )
+    (pin "11")
+    (pin "12")
+    (pin "14")
+    (pin "21")
+    (pin "22")
+    (pin "24")
+    (pin "A1")
+    (pin "A2")
+    (instances
+      (project "HWSRedirector"
+        (path "/4cdf1f0d-fc9e-401b-a9f3-d905b9fa1fb5"
+          (reference "K2") (unit 1)
+        )
+      )
+    )
+  )
+  (symbol (lib_id "Switch:SW_SPST") (at 78.74 119.38 270) (unit 1)
+    (in_bom yes) (on_board yes) (dnp no)
+    (property "Reference" "SW1" (at 81.153 118.7363 90)
+      (effects (font (size 1.27 1.27)) (justify left) hide)
+    )
+    (property "Value" "HWS Switch - May not be needed" (at 43.18 121.92 90) (do_not_autoplace)
+      (effects (font (size 1.27 1.27)) (justify left))
+    )
+    (property "Footprint" "" (at 78.74 119.38 0)
+      (effects (font (size 1.27 1.27)) hide)
+    )
+    (property "Datasheet" "~" (at 78.74 119.38 0)
       (effects (font (size 1.27 1.27)) hide)
     )
     (pin "1")
     (pin "2")
-    (pin "3")
-    (pin "4")
-    (pin "A1")
-    (pin "A2")
-    (instances
-      (project "HWSRedirector"
-        (path "/4cdf1f0d-fc9e-401b-a9f3-d905b9fa1fb5"
-          (reference "K2") (unit 1)
-        )
-      )
-    )
-  )
-  (symbol (lib_id "Switch:SW_SPST") (at 78.74 119.38 270) (unit 1)
-    (in_bom yes) (on_board yes) (dnp no)
-    (property "Reference" "SW1" (at 81.153 118.7363 90)
-      (effects (font (size 1.27 1.27)) (justify left) hide)
-    )
-    (property "Value" "HWS Switch" (at 66.064 119.3998 90) (do_not_autoplace)
-      (effects (font (size 1.27 1.27)) (justify left))
-    )
-    (property "Footprint" "" (at 78.74 119.38 0)
-      (effects (font (size 1.27 1.27)) hide)
-    )
-    (property "Datasheet" "~" (at 78.74 119.38 0)
-      (effects (font (size 1.27 1.27)) hide)
-    )
-    (pin "1")
-    (pin "2")
     (instances
       (project "HWSRedirector"
@@
     )
   )
-  (symbol (lib_id "HWS 2:Meter") (at 67.31 39.37 0) (unit 1)
-    (in_bom yes) (on_board yes) (dnp no)
-    (property "Reference" "U2" (at 76.727 53.8437 0)
+  (symbol (lib_id "HWS 2:Meter") (at 68.58 22.86 0) (unit 1)
+    (in_bom yes) (on_board yes) (dnp no)
+    (property "Reference" "U2" (at 77.997 37.3337 0)
       (effects (font (size 1.27 1.27)) (justify left) hide)
     )
-    (property "Value" "~" (at 67.31 39.37 0)
+    (property "Value" "~" (at 68.58 22.86 0)
       (effects (font (size 1.27 1.27)))
     )
-    (property "Footprint" "" (at 67.31 39.37 0)
-      (effects (font (size 1.27 1.27)) hide)
-    )
-    (property "Datasheet" "" (at 67.31 39.37 0)
+    (property "Footprint" "" (at 68.58 22.86 0)
+      (effects (font (size 1.27 1.27)) hide)
+    )
+    (property "Datasheet" "" (at 68.58 22.86 0)
       (effects (font (size 1.27 1.27)) hide)
     )
@@
       (effects (font (size 1.27 1.27)) (justify left))
     )
-    (property "Value" "WeMos C3" (at 179.9107 68.3146 0)
-      (effects (font (size 1.27 1.27)) (justify left))
-    )
+    (property "Value" "WeMos C3 or other WiFi Enabled ESP32" (at 179.9107 68.3146 0)
+      (effects (font (size 1.27 1.27)) (justify left))
+    )
